File: UAK_0/UAK_0.sch (KiCad schematic (older format))
At the start: 54 parts, among them K1 Кнопка_FSMSM, K2 Кнопка_FSMSM, X1 Крепежное_отверстие_М3, X2 Крепежное_отверстие_М3, X3 Крепежное_отверстие_М3, X4 Крепежное_отверстие_М3

Commit message: правки атрибутов УГО, заменен резистор RC-фильтра
Parts:
- R22: INFO 10 МОм -> 4,7 кОм
Changed lines of the file:
@@
 F 3 "" H 12500 3700 60  0001 C CNN
 F 4 "10 кОм" V 12550 3300 50  0000 L CNN "INFO"
-F 5 "" H 12500 3848 50  0001 C CNN "LINK"
 	1    12500 3700
 	0    -1   1    0
@@
 F 3 "" H 13000 3700 60  0001 C CNN
 F 4 "10 кОм" V 13050 3300 50  0000 L CNN "INFO"
-F 5 "" H 13000 3848 50  0001 C CNN "LINK"
 	1    13000 3700
 	0    -1   1    0
@@
 F 3 "" H 13800 4250 60  0001 C CNN
 F 4 "240 Ом" H 13700 4100 50  0000 L CNN "INFO"
-F 5 "" H 13800 4398 50  0001 C CNN "LINK"
 	1    13800 4250
 	-1   0    0    -1
@@
 F 3 "" H 13800 4750 60  0001 C CNN
 F 4 "240 Ом" H 13700 4600 50  0000 L CNN "INFO"
-F 5 "" H 13800 4898 50  0001 C CNN "LINK"
 	1    13800 4750
 	-1   0    0    -1
@@
 F 3 "" H 12550 7500 60  0001 C CNN
 F 4 "10 кОм" H 12400 7650 50  0000 L CNN "INFO"
-F 5 "" H 12550 7648 50  0001 C CNN "LINK"
 	1    12550 7500
 	1    0    0    1
@@
 F 3 "" H 13550 7500 60  0001 C CNN
 F 4 "240 Ом" H 13450 7350 50  0000 L CNN "INFO"
-F 5 "" H 13550 7648 50  0001 C CNN "LINK"
 	1    13550 7500
 	-1   0    0    -1
@@
 F 3 "" H 7950 2000 60  0001 C CNN
 F 4 "240 Ом" H 7850 1850 50  0000 L CNN "INFO"
-F 5 "" H 7950 2148 50  0001 C CNN "LINK"
 	1    7950 2000
 	-1   0    0    -1
@@
 F 3 "" H 9050 2500 60  0001 C CNN
 F 4 "10 кОм" H 8900 2650 50  0000 L CNN "INFO"
-F 5 "" H 9050 2648 50  0001 C CNN "LINK"
 	1    9050 2500
 	1    0    0    1
@@
 F 3 "" H 9000 7800 60  0001 C CNN
 F 4 "10 кОм" H 8850 7950 50  0000 L CNN "INFO"
-F 5 "" H 9000 7948 50  0001 C CNN "LINK"
 	1    9000 7800
 	1    0    0    1
@@
 F 3 "" H 7900 7300 60  0001 C CNN
 F 4 "240 Ом" H 7800 7150 50  0000 L CNN "INFO"
-F 5 "" H 7900 7448 50  0001 C CNN "LINK"
 	1    7900 7300
 	-1   0    0    -1
@@
 F 3 "" H 9050 4750 60  0001 C CNN
 F 4 "10 кОм" H 8900 4900 50  0000 L CNN "INFO"
-F 5 "" H 9050 4898 50  0001 C CNN "LINK"
 	1    9050 4750
 	1    0    0    1
@@
 F 3 "" H 7950 4250 60  0001 C CNN
 F 4 "240 Ом" H 7850 4100 50  0000 L CNN "INFO"
-F 5 "" H 7950 4398 50  0001 C CNN "LINK"
 	1    7950 4250
 	-1   0    0    -1
@@
 F 3 "" H 12550 9000 60  0001 C CNN
 F 4 "10 кОм" H 12400 9150 50  0000 L CNN "INFO"
-F 5 "" H 12550 9148 50  0001 C CNN "LINK"
 	1    12550 9000
 	1    0    0    1
@@
 F 3 "" H 13550 9000 60  0001 C CNN
 F 4 "240 Ом" H 13450 8850 50  0000 L CNN "INFO"
-F 5 "" H 13550 9148 50  0001 C CNN "LINK"
 	1    13550 9000
 	-1   0    0    -1
@@
 F 3 "" H 3400 5750 60  0001 C CNN
 F 4 "150 Ом" H 3300 5600 50  0000 L CNN "INFO"
-F 5 "" H 3400 5898 50  0001 C CNN "LINK"
 	1    3400 5750
 	-1   0    0    -1
@@
 F 3 "" H 3050 7150 60  0001 C CNN
 F 4 "10 кОм" H 2900 7300 50  0000 L CNN "INFO"
-F 5 "" H 3050 7298 50  0001 C CNN "LINK"
 	1    3050 7150
 	1    0    0    1
@@
 F 3 "" H 1950 6650 60  0001 C CNN
 F 4 "240 Ом" H 1850 6500 50  0000 L CNN "INFO"
-F 5 "" H 1950 6798 50  0001 C CNN "LINK"
 	1    1950 6650
 	-1   0    0    -1
@@
 F 2 "N_RLC:Резистор_SMD_1206-0,25_Вт" H 4750 6800 60  0001 C CNN
 F 3 "" H 4750 6800 60  0001 C CNN
-F 4 "10 МОм" V 4803 6903 50  0000 L CNN "INFO"
+F 4 "4,7 кОм" V 4803 6903 50  0000 L CNN "INFO"
 F 5 "https://www.chipdip.ru/product0/9000079814" H 4750 6800 50  0001 C CNN "LINK"
 	1    4750 6800

Commit message: UAK.1A.M9
исправлено межоснвое растояние крепежки экрана, заменен диод закольцовки зумера на сопротивление 4,7 кОм
Parts:
- removed VD2: Диод_шоттки_SK16, N_VD_HL:Диод_SMB, symbol UAK_0-rescue:Диод_шоттки_SK16-elements_2020
- added R23: Резистор_0,25Вт, N_RLC:Резистор_SMD_1206-0,25_Вт, symbol elements:Резистор_0,25Вт
Connections:
- net 5V: now also R23.1
- net at HA1.2, VT3.3: now also R23.2
Changed lines of the file:
@@
 encoding utf-8
 Sheet 1 2
-Title "UAK.0C.M9"
+Title "UAK.1A.M9"
 Date ""
 Rev ""
@@
 	1    0    0    -1
 $EndComp
-Text Label 10750 3850 0    50   ~ 0
-5V
 Wire Wire Line
 	11000 3850 10750 3850
@@
 	1    0    0    -1
 $EndComp
-Text Label 9750 3250 0    50   ~ 0
+Text Label 10750 3250 0    50   ~ 0
 5V
 Wire Notes Line
@@
 Connection ~ 9750 3950
 Wire Wire Line
-	9750 3750 9750 3950
-Wire Wire Line
-	9750 3250 9750 3450
-Wire Wire Line
 	9550 3950 9750 3950
-$Comp
-L UAK_0-rescue:Диод_шоттки_SK16-elements_2020 VD2
-U 1 1 5F5E6E89
-P 9750 3750
-F 0 "VD2" V 9950 3600 50  0000 C CNN
-F 1 "Диод_шоттки_SK16" V 9850 3300 50  0000 C CNN
-F 2 "N_VD_HL:Диод_SMB" H 9925 3525 50  0001 C CNN
-F 3 "https://static.chipdip.ru/lib/046/DOC003046730.pdf" H 9650 3750 50  0001 C CNN
-F 4 "1А, 60В" H 9925 3300 50  0001 C CNN "INFO"
-F 5 "https://www.chipdip.ru/product/sk16-diotec" H 9925 3425 50  0001 C CNN "LINK"
-	1    9750 3750
-	0    -1   -1   0
-$EndComp
 Text Label 10000 4750 2    50   ~ 0
 GND
@@
 Text Label 14500 9150 0    50   ~ 0
 GND
+$Comp
+L elements:Резистор_0,25Вт R23
+U 1 1 5F6845FD
+P 10300 3500
+F 0 "R23" H 10250 3350 60  0000 L CNN
+F 1 "Резистор_0,25Вт" H 10300 3350 60  0001 C CNN
+F 2 "N_RLC:Резистор_SMD_1206-0,25_Вт" H 10300 3500 60  0001 C CNN
+F 3 "" H 10300 3500 60  0001 C CNN
+F 4 "4,7 кОм" H 10150 3650 50  0000 L CNN "INFO"
+F 5 "https://www.chipdip.ru/product0/9000079814" H 10300 3500 50  0001 C CNN "LINK"
+	1    10300 3500
+	-1   0    0    1
+$EndComp
+Wire Wire Line
+	10000 3500 9750 3500
+Wire Wire Line
+	9750 3500 9750 3950
+Wire Wire Line
+	10600 3500 10750 3500
+Wire Wire Line
+	10750 3500 10750 3250
+Wire Wire Line
+	10750 3500 10750 3850
+Connection ~ 10750 3500
 $EndSCHEMATC

Commit message: ссылка на сайт заменена на лого
Parts:
- added D1: LOGO, N_ICO:bleeper_4x33, symbol elements:LOGO
Changed lines of the file:
@@
 	10750 3500 10750 3850
 Connection ~ 10750 3500
+$Comp
+L elements:LOGO D1
+U 1 1 5F6B4E2E
+P 9000 10500
+F 0 "D1" H 8925 10700 50  0001 C CNN
+F 1 "LOGO" H 8900 10500 50  0000 L CNN
+F 2 "N_ICO:bleeper_4x33" H 9000 10500 50  0001 C CNN
+F 3 "" H 9000 10500 50  0001 C CNN
+	1    9000 10500
+	1    0    0    -1
+$EndComp
 $EndSCHEMATC
