File: UAK_0/UAK_0.kicad_pcb (KiCad board)
At the start: 2 copper layers, 100 x 90 mm, 79 parts, among them K1 Кнопка_FSMSM, K2 Кнопка_FSMSM, X1 Крепежное_отверстие_М3, X2 Крепежное_отверстие_М3, X3 Крепежное_отверстие_М3, X4 Крепежное_отверстие_М3, X5 Крепежное_отверстие_d2, X6 Крепежное_отверстие_d2, X7 Крепежное_отверстие_d2

Commit message: ссылка на сайт заменена на лого
Parts:
- added D1: LOGO, N_ICO:bleeper_4x33, B.Cu at (114.8, 68.5)
Other:
- board text removed: "WWW.BLEEPER.RU"

Commit message: исправлено лого bleeper, исправлено место зуммера
Routing:
- net Net-(HA1-Pad2): track 17.9 -> 21.4 mm
- net /5V: track 306.7 -> 309.8 mm

Commit message: обновлены 3D в проекте и step
Other:
- board text added: "UAK.0C_M.M9"
- board text removed: "UAK.1A.M9"
