File: UAK_1/UAK_1.sch (KiCad schematic (older format))
At the start: 55 parts, among them K1 Кнопка_FSMSM, K2 Кнопка_FSMSM, X1 Крепежное_отверстие_М3, X2 Крепежное_отверстие_М3, X3 Крепежное_отверстие_М3, X4 Крепежное_отверстие_М3

Commit message: 1B: заменены предохранители,обновлено питание,не добавлен второй дисплей
Parts:
- removed FU2: Предохранитель, N_RLC:Предохранитель_SMD_1812, symbol elements:Предохранитель
- removed XT5: Клеммник_х2_KLS2-300-5.00-02P-2S, N_X:Клеммник_х2_шаг5, symbol UAK_1-rescue:Клеммник_х2_KLS2-300-5.00-02P-2S-elements_2020-UAK_0-rescue
- added XFU1, XFU2: Держатель_предохранителя_KLS5-266, N_X:Держатель_5х20, symbol elements_2020:Держатель_предохранителя_KLS5-266
Connections:
- net labels added: 220_L_FU
- net labels removed: 0V_RES, 12V_RES, 220_N_FU
- wire segments 182 -> 180
Other:
- moved on the sheet: XT4
Changed lines of the file:
@@
 EESchema Schematic File Version 4
 LIBS:UAK_1-cache
-EELAYER 29 0
+EELAYER 30 0
 EELAYER END
 $Descr A3 16535 11693
@@
 L UAK_1-rescue:Клеммник_х2_KLS2-300-5.00-02P-2S-elements_2020-UAK_0-rescue XT4
 U 1 1 5F53E542
-P 14500 1500
-F 0 "XT4" H 14150 1850 60  0000 L CNN
-F 1 "Клеммник_х2_KLS2-300-5.00-02P-2S" H 14190 1240 60  0001 C CNN
-F 2 "N_X:Клеммник_х2_шаг5" H 13925 1775 60  0001 C CNN
-F 3 "" H 13925 1775 60  0001 C CNN
-	1    14500 1500
-	-1   0    0    -1
-$EndComp
-Text Label 14500 1500 0    50   ~ 0
+P 14750 1500
+F 0 "XT4" H 14400 1850 60  0000 L CNN
+F 1 "Клеммник_х2_KLS2-300-5.00-02P-2S" H 14440 1240 60  0001 C CNN
+F 2 "N_X:Клеммник_х2_шаг5" H 14175 1775 60  0001 C CNN
+F 3 "" H 14175 1775 60  0001 C CNN
+	1    14750 1500
+	-1   0    0    -1
+$EndComp
+Text Label 14750 1500 0    50   ~ 0
 220_L
-Text Label 14500 1650 0    50   ~ 0
+Text Label 14750 1650 0    50   ~ 0
 220_N
 $Sheet
-S 13000 1250 1000 1250
+S 12250 1250 1000 1250
 U 5F540B17
 F0 "SUPPLY_POWER" 50
 F1 "SUPPLY_POWER.sch" 50
-F2 "220_L" I R 14000 1500 50
-F3 "220_N" I R 14000 1750 50
-F4 "GND" I L 13000 2250 50
-F5 "3V3" I L 13000 2000 50
-F6 "5V" I L 13000 1750 50
-F7 "12V" I L 13000 1500 50
-F8 "12V_RESERV" I R 14000 2400 50
-F9 "0V_RESERV" I R 14000 2250 50
+F2 "220_L" I R 13250 1500 50
+F3 "220_N" I R 13250 1750 50
+F4 "GND" I L 12250 2250 50
+F5 "3V3" I L 12250 2000 50
+F6 "5V" I L 12250 1750 50
+F7 "12V" I L 12250 1500 50
 $EndSheet
-Wire Wire Line
-	14000 1500 14500 1500
-Wire Wire Line
-	14000 1750 14250 1750
-Wire Wire Line
-	14250 1750 14250 1650
-Wire Wire Line
-	14250 1650 14500 1650
 Text Label 1000 1300 0    50   ~ 0
 EN_RESET
@@
 	1500 1300 1000 1300
 Wire Wire Line
-	13000 2000 12500 2000
-Wire Wire Line
-	13000 2250 12500 2250
-Text Label 12500 2250 0    50   ~ 0
-GND
-Text Label 12500 2000 0    50   ~ 0
+	12250 2000 12000 2000
+Wire Wire Line
+	12250 2250 12000 2250
+Text Label 12000 2250 0    50   ~ 0
+GND
+Text Label 12000 2000 0    50   ~ 0
 3V3
 Text Label 1000 1000 0    50   ~ 0
@@
 $EndComp
 Wire Wire Line
-	13000 1500 12500 1500
-Text Label 12500 1500 0    50   ~ 0
+	12250 1500 12000 1500
+Text Label 12000 1500 0    50   ~ 0
 12V
 Text Label 10750 1550 0    50   ~ 0
@@
 	11500 2750 11500 750
 Wire Wire Line
-	13000 1750 12500 1750
-Text Label 12500 1750 0    50   ~ 0
+	12250 1750 12000 1750
+Text Label 12000 1750 0    50   ~ 0
 5V
 Text Label 5500 1850 2    50   ~ 0
@@
 НА СВЕТОДИОДНУЮ ЛЕНТУ WS2812
 $Comp
-L UAK_1-rescue:Клеммник_х2_KLS2-300-5.00-02P-2S-elements_2020-UAK_0-rescue XT5
-U 1 1 5F82F0A6
-P 14500 2250
-F 0 "XT5" H 14150 2600 60  0000 L CNN
-F 1 "Клеммник_х2_KLS2-300-5.00-02P-2S" H 14190 1990 60  0001 C CNN
-F 2 "N_X:Клеммник_х2_шаг5" H 13925 2525 60  0001 C CNN
-F 3 "" H 13925 2525 60  0001 C CNN
-	1    14500 2250
-	-1   0    0    -1
-$EndComp
-Wire Wire Line
-	14000 2250 14500 2250
-Wire Wire Line
-	14000 2400 14500 2400
-Text Label 14500 2400 0    50   ~ 0
-12V_RES
-Text Label 14500 2250 0    50   ~ 0
-0V_RES
-$Comp
-L elements:Предохранитель FU2
-U 1 1 5F560616
-P 5600 5900
-AR Path="/5F560616" Ref="FU2"  Part="1"
-AR Path="/5F540B17/5F560616" Ref="FU?"  Part="1"
-F 0 "FU2" H 5600 6050 60  0000 C CNN
-F 1 "Предохранитель" H 5600 5750 60  0001 C CNN
-F 2 "N_RLC:Предохранитель_SMD_1812" H 5600 5900 60  0001 C CNN
-F 3 "" H 5600 5900 60  0001 C CNN
-F 4 "0,1А, 1812" H 5600 5750 50  0000 C CNN "INFO"
-F 5 "https://www.chipdip.ru/product/mf-msmf010" H 5600 5900 50  0001 C CNN "LINK"
-	1    5600 5900
-	1    0    0    -1
-$EndComp
-$Comp
 L UAK_1-rescue:Клеммник_х2_KLS2-300-5.00-02P-2S-elements_2020-UAK_0-rescue XT8
 U 1 1 5F5696D9
@@
 	-1   0    0    -1
 $EndComp
-Text Label 5750 7150 0    50   ~ 0
-220_L
 $Comp
 L UAK_1-rescue:МОП-реле_КР293КП1Б-elements_2020-UAK_0-rescue DA1
@@
 	1    0    0    1
 $EndComp
-Text Label 5000 5600 2    50   ~ 0
+Text Label 5250 5600 2    50   ~ 0
 220_N
 NoConn ~ 4700 5750
 NoConn ~ 4000 5600
-Text Label 6500 5900 2    50   ~ 0
+Text Label 5250 5900 2    50   ~ 0
 220_N_OUT
 Text Label 5750 7000 0    50   ~ 0
@@
 3V3
 Wire Wire Line
-	4700 5600 5000 5600
-Wire Wire Line
-	6000 5900 6500 5900
-Text Label 5100 5900 2    50   ~ 0
-220_N_FU
-Wire Wire Line
-	4700 5900 5200 5900
+	4700 5600 5250 5600
+Wire Wire Line
+	4700 5900 5250 5900
 Text Label 14500 7650 0    50   ~ 0
 GND
@@
 Text Label 10750 2400 0    50   ~ 0
 5V
+$Comp
+L elements_2020:Держатель_предохранителя_KLS5-266 XFU1
+U 1 1 5F802810
+P 13750 1500
+F 0 "XFU1" H 13800 1650 50  0000 L CNN
+F 1 "Держатель_предохранителя_KLS5-266" H 13850 1250 50  0001 C CNN
+F 2 "N_X:Держатель_5х20" H 13750 1500 50  0001 C CNN
+F 3 "" H 13750 1500 50  0001 C CNN
+F 4 "https://www.chipdip.ru/product/kls5-266-fh-100" H 13900 1175 50  0001 C CNN "LINK"
+	1    13750 1500
+	1    0    0    -1
+$EndComp
+$Comp
+L elements_2020:Держатель_предохранителя_KLS5-266 XFU2
+U 1 1 5F8032F7
+P 14500 1500
+F 0 "XFU2" H 14550 1650 50  0000 L CNN
+F 1 "Держатель_предохранителя_KLS5-266" H 14600 1250 50  0001 C CNN
+F 2 "N_X:Держатель_5х20" H 14500 1500 50  0001 C CNN
+F 3 "" H 14500 1500 50  0001 C CNN
+F 4 "https://www.chipdip.ru/product/kls5-266-fh-100" H 14650 1175 50  0001 C CNN "LINK"
+	1    14500 1500
+	-1   0    0    -1
+$EndComp
+Wire Wire Line
+	14500 1500 14750 1500
+Wire Wire Line
+	14500 1750 14500 1650
+Wire Wire Line
+	14500 1650 14750 1650
+Text Label 13350 1500 0    50   ~ 0
+220_L_FU
+Wire Wire Line
+	13250 1500 13750 1500
+Wire Wire Line
+	13250 1750 14500 1750
+Text Label 5750 7150 0    50   ~ 0
+220_L_FU
 $EndSCHEMATC

Commit message: обновлен перечень элементов
Parts:
- added D2: LOGO, N_ICO:danger_220, symbol elements:LOGO
- added XS1: Розетка_СНП346-16РП21-1-В, symbol MOTOR:Розетка_СНП346-16РП21-1-В
- A1: LINK (none) -> https://www.terraelectronica.ru/product/2292549; Для заказа (none) -> ESP32-WROOM-32 [4MB]
- C1, C3, C4, C5, C6: LINK https://www.chipdip.ru/product0/226236018 -> https://www.terraelectronica.ru/product/1044009; Для заказа (none) -> Конденсатор 0603 100 нФ 50В 5%
- C17: Для заказа (none) -> Конденсатор 1210 0,022 мкФ 630В 10%
- C2: LINK https://www.chipdip.ru/product0/101260414 -> https://www.terraelectronica.ru/product/363479; Для заказа (none) -> Конденсатор D 100 мкФ 10В 20%
- D1: INFO (none) -> PCB_element; Для заказа (none) -> -
- DA1: Для заказа (none) -> МОП-реле КР293КП1Б
- DD1: LINK https://www.chipdip.ru/product/mc74vhc1gt125dt1g -> https://www.terraelectronica.ru/product/274803; Для заказа (none) -> Повторитель M74VHC1GT125DF2G
- HA1: Для заказа (none) -> Зуммер HPA17F
- HL1, X1, X2, X3, X4: Для заказа (none) -> -
- K1, K2: LINK https://www.chipdip.ru/product/tyco-1437566-3-fsmsm -> https://www.terraelectronica.ru/product/1087727; Для заказа (none) -> Кнопка FSMSM
- R1, R11, R12, R13, R14, R19, R2, R3: LINK (none) -> https://www.terraelectronica.ru/product/559067; Для заказа (none) -> Резистор 0603 240 Ом 5%
- R10, R20, R4, R5, R6, R7, R8, R9: LINK (none) -> https://www.terraelectronica.ru/product/562124; Для заказа (none) -> Резистор 0603 10 кОм 5%
- R21: LINK (none) -> https://www.terraelectronica.ru/product/569439; Для заказа (none) -> Резистор 0603 150 Ом 5%
- R22, R23: LINK https://www.chipdip.ru/product0/9000079814 -> https://www.terraelectronica.ru/product/2782734; Для заказа (none) -> Резистор 1206 4,7 кОм 5%
- RP1: LINK https://www.chipdip.ru/product/3303x-3-103 -> https://www.chipdip.ru/product/3303x-3-503; Для заказа (none) -> Резистор подстроечный 50 кОм
- VD1: LINK https://www.chipdip.ru/product/sk16-diotec -> https://www.terraelectronica.ru/product/129173; Для заказа (none) -> Диод шоттки SK16 (1А 60В)
- VD3: LINK https://www.chipdip.ru/product/bar43cfilm -> https://www.terraelectronica.ru/product/296487; Для заказа (none) -> Набор диодов BAR43CFILM
- VT1, VT2, VT3, VT4: Для заказа (none) -> Транзистор N-канал IRLML6344TRPBF
- XFU1, XFU2: Для заказа (none) -> Держатель KLS5-266
- XP1: Для заказа (none) -> Вилка угловая WF-4R
- XT1, XT2, XT3, XT6, XT7: Для заказа (none) -> Клеммник 308-021-14 (шаг 2,54 мм)
- XT4, XT8: LINK (none) -> https://www.chipdip.ru/product/kls2-300-5.00-02p-2s-dg300-5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; Для заказа (none) -> Клеммник KLS2-300-5.00-02P-2S (шаг 5 мм)
Connections:
- net DOOR_SENSOR: now also A1.28 (IO17); no longer A1.37 (IO23)
- new net MOSI: A1.37 (IO23)
- no-connect marks 6 -> 5

Commit message: UAK.1C.M9, подготовлены gerber, схема, BOM
обновлена маркировка, заполнен BOM
Parts:
- removed XS1: Розетка_СНП346-16РП21-1-В, symbol MOTOR:Розетка_СНП346-16РП21-1-В
- D1, D2, HL1, X1, X2, X3, X4: LINK (none) -> -
- XFU1, XFU2: symbol elements_2020:Держатель_предохранителя_KLS5-266 -> UAK_1-rescue:Держатель_предохранителя_KLS5-266-elements_2020
Changed lines of the file:
@@
 EESchema Schematic File Version 4
 LIBS:UAK_1-cache
-EELAYER 30 0
+EELAYER 29 0
 EELAYER END
 $Descr A3 16535 11693
 encoding utf-8
 Sheet 1 2
-Title "UAK.1A.M9"
+Title "UAK.1C.M9"
 Date ""
 Rev ""
@@
 F 4 "PCB_element" H 11000 10300 50  0001 C CNN "INFO"
 F 5 "-" H 11000 10500 50  0001 C CNN "Для заказа"
+F 6 "-" H 11000 10500 50  0001 C CNN "LINK"
 	1    11000 10500
 	1    0    0    -1
@@
 F 4 "PCB_element" H 10500 10300 50  0001 C CNN "INFO"
 F 5 "-" H 10500 10500 50  0001 C CNN "Для заказа"
+F 6 "-" H 10500 10500 50  0001 C CNN "LINK"
 	1    10500 10500
 	1    0    0    -1
@@
 F 4 "PCB_element" H 10000 10300 50  0001 C CNN "INFO"
 F 5 "-" H 10000 10500 50  0001 C CNN "Для заказа"
+F 6 "-" H 10000 10500 50  0001 C CNN "LINK"
 	1    10000 10500
 	1    0    0    -1
@@
 F 4 "PCB_element" H 9500 10300 50  0001 C CNN "INFO"
 F 5 "-" H 9500 10500 50  0001 C CNN "Для заказа"
+F 6 "-" H 9500 10500 50  0001 C CNN "LINK"
 	1    9500 10500
 	1    0    0    -1
@@
 F 3 "http://www.melt.com.ru/docs/MT-16S2H.pdf" H 10000 5500 50  0001 C CNN
 F 4 "-" H 10000 5500 50  0001 C CNN "Для заказа"
+F 5 "-" H 10000 5500 50  0001 C CNN "LINK"
 	1    10000 5500
 	1    0    0    -1
@@
 F 4 "PCB_element" H 9000 10500 50  0001 C CNN "INFO"
 F 5 "-" H 9000 10500 50  0001 C CNN "Для заказа"
+F 6 "-" H 9000 10500 50  0001 C CNN "LINK"
 	1    9000 10500
 	1    0    0    -1
@@
 5V
 $Comp
-L elements_2020:Держатель_предохранителя_KLS5-266 XFU1
+L UAK_1-rescue:Держатель_предохранителя_KLS5-266-elements_2020 XFU1
 U 1 1 5F802810
 P 13750 1500
@@
 $EndComp
 $Comp
-L elements_2020:Держатель_предохранителя_KLS5-266 XFU2
+L UAK_1-rescue:Держатель_предохранителя_KLS5-266-elements_2020 XFU2
 U 1 1 5F8032F7
 P 14500 1500
@@
 F 4 "PCB_element" H 8500 10500 50  0001 C CNN "INFO"
 F 5 "-" H 8500 10500 50  0001 C CNN "Для заказа"
+F 6 "-" H 8500 10500 50  0001 C CNN "LINK"
 	1    8500 10500
 	1    0    0    -1
@@
 Text Label 6000 1250 2    50   ~ 0
 MOSI
-$Comp
-L MOTOR:Розетка_СНП346-16РП21-1-В XS1
-U 1 1 5F9C70A1
-P 5250 8550
-F 0 "XS1" H 5508 8737 60  0000 C CNN
-F 1 "Розетка_СНП346-16РП21-1-В" H 5508 8631 60  0000 C CNN
-F 2 "" H 5250 8550 60  0001 C CNN
-F 3 "" H 5250 8550 60  0001 C CNN
-F 4 "https://www.chipdip.ru/product/pbs16" H 5250 8550 50  0001 C CNN "LINK"
-F 5 "Розетка PBS-16" H 5250 8550 50  0001 C CNN "Для заказа"
-	1    5250 8550
-	1    0    0    -1
-$EndComp
 $EndSCHEMATC
