File: UAK_2/SUPPLY_POWER.sch (KiCad schematic (older format))
At the start: 17 parts

Commit message: добавлена методика программирования, на схему вынесен новый дисплей
Parts:
- G1: symbol UAK_1-rescue:AC-DC-преобразователь_IRM-15-5-elements_2020 -> UAK_2-rescue:AC-DC-преобразователь_IRM-15-5-elements_2020-UAK_1-rescue
- L1: symbol UAK_1-rescue:Чип-индуктивность_10мкГн_1.8А_20проц.-elements_2020-UAK_0-rescue -> UAK_2-rescue:Чип-индуктивность_10мкГн_1.8А_20проц.-elements_2020-UAK_0-rescue-UAK_1-rescue
- L2: symbol UAK_1-rescue:Дроссель_B82731-T2132-A20_2х6.8мГн_1.3А_250В-elements_2020-UAK_0-rescue -> UAK_2-rescue:Дроссель_B82731-T2132-A20_2х6.8мГн_1.3А_250В-elements_2020-UAK_0-rescue-UAK_1-rescue
- VD2: symbol UAK_1-rescue:Диод_шоттки_SK16-elements_2020-UAK_0-rescue -> UAK_2-rescue:Диод_шоттки_SK16-elements_2020-UAK_0-rescue-UAK_1-rescue
Changed lines of the file:
@@
 EESchema Schematic File Version 4
-LIBS:UAK_1-cache
+LIBS:UAK_2-cache
 EELAYER 29 0
 EELAYER END
@@
 	6250 1600 6250 1500
 $Comp
-L UAK_1-rescue:Дроссель_B82731-T2132-A20_2х6.8мГн_1.3А_250В-elements_2020-UAK_0-rescue L2
+L UAK_2-rescue:Дроссель_B82731-T2132-A20_2х6.8мГн_1.3А_250В-elements_2020-UAK_0-rescue-UAK_1-rescue L2
 U 1 1 5F5455B1
 P 7250 1600
@@
 5V_NOISE
 $Comp
-L UAK_1-rescue:AC-DC-преобразователь_IRM-15-5-elements_2020 G1
+L UAK_2-rescue:AC-DC-преобразователь_IRM-15-5-elements_2020-UAK_1-rescue G1
 U 1 1 5F6F4DEB
 P 4300 1500
@@
 $EndComp
 $Comp
-L UAK_1-rescue:Чип-индуктивность_10мкГн_1.8А_20проц.-elements_2020-UAK_0-rescue L1
+L UAK_2-rescue:Чип-индуктивность_10мкГн_1.8А_20проц.-elements_2020-UAK_0-rescue-UAK_1-rescue L1
 U 1 1 5F70E05E
 P 5550 3000
@@
 $EndComp
 $Comp
-L UAK_1-rescue:Диод_шоттки_SK16-elements_2020-UAK_0-rescue VD?
+L UAK_2-rescue:Диод_шоттки_SK16-elements_2020-UAK_0-rescue-UAK_1-rescue VD?
 U 1 1 5F71D917
 P 6750 3000
