File: UAK_3/SUPPLY_POWER.sch (KiCad schematic (older format))
At the start: 8 parts

Commit message: BOM переопределен по всему, кроме резисторов
Parts:
- C10: LCSC (none) -> C304015; LINK https://www.chipdip.ru/product/grm32qr72j223k -> https://lcsc.com/product-detail/Multilayer-Ceramic-Capacito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
- C12, C13, C15, C16: INFO 10мкФ/25В -> 10мкФ/10В; LCSC (none) -> C19702; LINK https://www.terraelectronica.ru/product/1489875 -> https://lcsc.com/product-detail/Multilayer-Ceramic-Capacito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
- G1, L2: LCSC (none) -> -
- G2: LCSC (none) -> C173386; LINK https://www.chipdip.ru/product/lm1117gs-3.3 -> https://lcsc.com/product-detail/Dropout-Regulators-LDO_Shen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
Changed lines of the file:
@@
 EESchema Schematic File Version 4
 LIBS:UAK_3-cache
-EELAYER 30 0
+EELAYER 29 0
 EELAYER END
 $Descr A4 11693 8268
@@
 F 3 "" H 3250 1700 60  0001 C CNN
 F 4 "0,022мкФ/630В" V 3328 1788 50  0000 L CNN "INFO"
-F 5 "https://www.chipdip.ru/product/grm32qr72j223k" H 3250 1700 50  0001 C CNN "LINK"
+F 5 "https://lcsc.com/product-detail/Multilayer-Ceramic-Capacitors-MLCC-SMD-SMT_Walsin-Tech-Corp-1210B223K102CT_C304015.html/?href=jlc-SMT" H 3250 1700 50  0001 C CNN "LINK"
 F 6 "Конденсатор 1210 0,022 мкФ 630В 10%" H 3250 1700 50  0001 C CNN "Для заказа"
+F 7 "C304015 " H 3250 1700 50  0001 C CNN "LCSC"
 	1    3250 1700
 	0    1    1    0
@@
 F 2 "N_RLC:Конденсатор_SMD_0603" H 6250 1650 60  0001 C CNN
 F 3 "" H 6250 1650 60  0001 C CNN
-F 4 "10мкФ/25В" V 6328 1738 50  0000 L CNN "INFO"
-F 5 "https://www.terraelectronica.ru/product/1489875" H 6250 1650 50  0001 C CNN "LINK"
+F 4 "10мкФ/10В" V 6328 1738 50  0000 L CNN "INFO"
+F 5 "https://lcsc.com/product-detail/Multilayer-Ceramic-Capacitors-MLCC-SMD-SMT_Samsung-Electro-Mechanics-CL10A106KP8NNNC_C19702.html/?href=jlc-SMT" H 6250 1650 50  0001 C CNN "LINK"
 F 6 "Конденсатор 0603 10 мкФ 25В 20%" H 6250 1650 50  0001 C CNN "Для заказа"
+F 7 "C19702 " H 6250 1650 50  0001 C CNN "LCSC"
 	1    6250 1650
 	0    1    1    0
@@
 F 5 "2x6,8мГн/1,3А" V 7450 1650 50  0000 L CNN "INFO"
 F 6 "Дроссель B82731-T2132-A20" H 7250 1600 50  0001 C CNN "Для заказа"
+F 7 "-" H 7250 1600 50  0001 C CNN "LCSC"
 	1    7250 1600
 	0    1    1    0
@@
 F 2 "N_RLC:Конденсатор_SMD_0603" H 8000 1650 60  0001 C CNN
 F 3 "" H 8000 1650 60  0001 C CNN
-F 4 "10мкФ/25В" V 8078 1738 50  0000 L CNN "INFO"
-F 5 "https://www.terraelectronica.ru/product/1489875" H 8000 1650 50  0001 C CNN "LINK"
+F 4 "10мкФ/10В" V 8078 1738 50  0000 L CNN "INFO"
+F 5 "https://lcsc.com/product-detail/Multilayer-Ceramic-Capacitors-MLCC-SMD-SMT_Samsung-Electro-Mechanics-CL10A106KP8NNNC_C19702.html/?href=jlc-SMT" H 8000 1650 50  0001 C CNN "LINK"
 F 6 "Конденсатор 0603 10 мкФ 25В 20%" H 8000 1650 50  0001 C CNN "Для заказа"
+F 7 "C19702 " H 8000 1650 50  0001 C CNN "LCSC"
 	1    8000 1650
 	0    1    1    0
@@
 F 2 "N_VD_HL:Транзистор_NPN_SOT223" H 4550 6000 50  0001 C CNN
 F 3 "https://static.chipdip.ru/lib/138/DOC004138838.pdf" H 4550 6000 50  0001 C CNN
-F 4 "https://www.chipdip.ru/product/lm1117gs-3.3" H 4550 6000 50  0001 C CNN "LINK"
+F 4 "https://lcsc.com/product-detail/Dropout-Regulators-LDO_Shenzhen-Fuman-Elec-SC1117-3-3V_C173386.html/?href=jlc-SMT" H 4550 6000 50  0001 C CNN "LINK"
 F 5 "LDO LM1117GS-3.3" H 4550 6000 50  0001 C CNN "Для заказа"
+F 6 "C173386 " H 4550 6000 50  0001 C CNN "LCSC"
 	1    4550 6000
 	1    0    0    -1
@@
 F 2 "N_RLC:Конденсатор_SMD_0603" H 4000 6150 60  0001 C CNN
 F 3 "" H 4000 6150 60  0001 C CNN
-F 4 "10мкФ/25В" V 4078 6238 50  0000 L CNN "INFO"
-F 5 "https://www.terraelectronica.ru/product/1489875" H 4000 6150 50  0001 C CNN "LINK"
+F 4 "10мкФ/10В" V 4078 6238 50  0000 L CNN "INFO"
+F 5 "https://lcsc.com/product-detail/Multilayer-Ceramic-Capacitors-MLCC-SMD-SMT_Samsung-Electro-Mechanics-CL10A106KP8NNNC_C19702.html/?href=jlc-SMT" H 4000 6150 50  0001 C CNN "LINK"
 F 6 "Конденсатор 0603 10 мкФ 25В 20%" H 4000 6150 50  0001 C CNN "Для заказа"
+F 7 "C19702 " H 4000 6150 50  0001 C CNN "LCSC"
 	1    4000 6150
 	0    1    1    0
@@
 F 2 "N_RLC:Конденсатор_SMD_0603" H 5500 6150 60  0001 C CNN
 F 3 "" H 5500 6150 60  0001 C CNN
-F 4 "10мкФ/25В" V 5578 6238 50  0000 L CNN "INFO"
-F 5 "https://www.terraelectronica.ru/product/1489875" H 5500 6150 50  0001 C CNN "LINK"
+F 4 "10мкФ/10В" V 5578 6238 50  0000 L CNN "INFO"
+F 5 "https://lcsc.com/product-detail/Multilayer-Ceramic-Capacitors-MLCC-SMD-SMT_Samsung-Electro-Mechanics-CL10A106KP8NNNC_C19702.html/?href=jlc-SMT" H 5500 6150 50  0001 C CNN "LINK"
 F 6 "Конденсатор 0603 10 мкФ 25В 20%" H 5500 6150 50  0001 C CNN "Для заказа"
+F 7 "C19702 " H 5500 6150 50  0001 C CNN "LCSC"
 	1    5500 6150
 	0    1    1    0
@@
 F 5 "220В/5В" H 4650 1300 50  0000 C CNN "INFO"
 F 6 "AC-DC IRM-15-5" H 4300 1500 50  0001 C CNN "Для заказа"
+F 7 "-" H 4300 1500 50  0001 C CNN "LCSC"
 	1    4300 1500
 	1    0    0    -1
