File: UAK_3/SUPPLY_POWER.sch (KiCad schematic (older format))
At the start: 8 parts

Commit message: подготовлены файлы для заказа в JLCPCB
Parts:
- C10: renamed from C13; footprint N_RLC:Конденсатор_SMD_0603 -> N_RLC:Конденсатор_SMD_0603_pnp
- C11: renamed from C16; footprint N_RLC:Конденсатор_SMD_0603 -> N_RLC:Конденсатор_SMD_0603_pnp
- C7: renamed from C10; footprint N_RLC:Конденсатор_SMD_1210 -> N_RLC:Конденсатор_SMD_1210_pnp
- C8: renamed from C12; footprint N_RLC:Конденсатор_SMD_0603 -> N_RLC:Конденсатор_SMD_0603_pnp
- C9: renamed from C15; footprint N_RLC:Конденсатор_SMD_0603 -> N_RLC:Конденсатор_SMD_0603_pnp
- G2: footprint N_VD_HL:Транзистор_NPN_SOT223 -> N_VD_HL:Транзистор_NPN_SOT223_pnp
- renumbered L2 to L1
Changed lines of the file:
@@
 P 3250 1700
 AR Path="/5F542189" Ref="C?"  Part="1"
-AR Path="/5F540B17/5F542189" Ref="C10"  Part="1"
-F 0 "C10" V 3230 1788 60  0000 L CNN
+AR Path="/5F540B17/5F542189" Ref="C7"  Part="1"
+F 0 "C7" V 3230 1788 60  0000 L CNN
 F 1 "Конденсатор_керамический" H 3350 1600 60  0001 C CNN
-F 2 "N_RLC:Конденсатор_SMD_1210" H 3250 1700 60  0001 C CNN
+F 2 "N_RLC:Конденсатор_SMD_1210_pnp" H 3250 1700 60  0001 C CNN
 F 3 "" H 3250 1700 60  0001 C CNN
 F 4 "0,022мкФ/630В" V 3328 1788 50  0000 L CNN "INFO"
@@
 P 6250 1650
 AR Path="/5F542191" Ref="C?"  Part="1"
-AR Path="/5F540B17/5F542191" Ref="C13"  Part="1"
-F 0 "C13" V 6230 1738 60  0000 L CNN
+AR Path="/5F540B17/5F542191" Ref="C10"  Part="1"
+F 0 "C10" V 6230 1738 60  0000 L CNN
 F 1 "Конденсатор_керамический" H 6350 1550 60  0001 C CNN
-F 2 "N_RLC:Конденсатор_SMD_0603" H 6250 1650 60  0001 C CNN
+F 2 "N_RLC:Конденсатор_SMD_0603_pnp" H 6250 1650 60  0001 C CNN
 F 3 "" H 6250 1650 60  0001 C CNN
 F 4 "10мкФ/10В" V 6328 1738 50  0000 L CNN "INFO"
@@
 	6250 1600 6250 1500
 $Comp
-L UAK_3-rescue:Дроссель_B82731-T2132-A20_2х6.8мГн_1.3А_250В-elements_2020-UAK_0-rescue-UAK_1-rescue-UAK_2-rescue L2
+L UAK_3-rescue:Дроссель_B82731-T2132-A20_2х6.8мГн_1.3А_250В-elements_2020-UAK_0-rescue-UAK_1-rescue-UAK_2-rescue L1
 U 1 1 5F5455B1
 P 7250 1600
-F 0 "L2" V 7250 1650 50  0000 L CNN
+F 0 "L1" V 7250 1650 50  0000 L CNN
 F 1 "Дроссель_B82731-T2132-A20_2х6.8мГн_1.3А_250В" V 7420 1688 50  0001 L CNN
 F 2 "N_RLC:Дроссель_B82731" V 7340 1410 50  0001 C CNN
@@
 P 8000 1650
 AR Path="/5F54B79E" Ref="C?"  Part="1"
-AR Path="/5F540B17/5F54B79E" Ref="C16"  Part="1"
-F 0 "C16" V 7980 1738 60  0000 L CNN
+AR Path="/5F540B17/5F54B79E" Ref="C11"  Part="1"
+F 0 "C11" V 7980 1738 60  0000 L CNN
 F 1 "Конденсатор_керамический" H 8100 1550 60  0001 C CNN
-F 2 "N_RLC:Конденсатор_SMD_0603" H 8000 1650 60  0001 C CNN
+F 2 "N_RLC:Конденсатор_SMD_0603_pnp" H 8000 1650 60  0001 C CNN
 F 3 "" H 8000 1650 60  0001 C CNN
 F 4 "10мкФ/10В" V 8078 1738 50  0000 L CNN "INFO"
@@
 F 0 "G2" H 4900 6265 50  0000 C CNN
 F 1 "стабилизатор_нерегулируемый_LM1117GS-3.3" H 4900 6174 50  0000 C CNN
-F 2 "N_VD_HL:Транзистор_NPN_SOT223" H 4550 6000 50  0001 C CNN
+F 2 "N_VD_HL:Транзистор_NPN_SOT223_pnp" H 4550 6000 50  0001 C CNN
 F 3 "https://static.chipdip.ru/lib/138/DOC004138838.pdf" H 4550 6000 50  0001 C CNN
 F 4 "https://lcsc.com/product-detail/Dropout-Regulators-LDO_Shenzhen-Fuman-Elec-SC1117-3-3V_C173386.html/?href=jlc-SMT" H 4550 6000 50  0001 C CNN "LINK"
@@
 P 4000 6150
 AR Path="/5F5A914F" Ref="C?"  Part="1"
-AR Path="/5F540B17/5F5A914F" Ref="C12"  Part="1"
-F 0 "C12" V 3980 6238 60  0000 L CNN
+AR Path="/5F540B17/5F5A914F" Ref="C8"  Part="1"
+F 0 "C8" V 3980 6238 60  0000 L CNN
 F 1 "Конденсатор_керамический" H 4100 6050 60  0001 C CNN
-F 2 "N_RLC:Конденсатор_SMD_0603" H 4000 6150 60  0001 C CNN
+F 2 "N_RLC:Конденсатор_SMD_0603_pnp" H 4000 6150 60  0001 C CNN
 F 3 "" H 4000 6150 60  0001 C CNN
 F 4 "10мкФ/10В" V 4078 6238 50  0000 L CNN "INFO"
@@
 P 5500 6150
 AR Path="/5F5AA72C" Ref="C?"  Part="1"
-AR Path="/5F540B17/5F5AA72C" Ref="C15"  Part="1"
-F 0 "C15" V 5480 6238 60  0000 L CNN
+AR Path="/5F540B17/5F5AA72C" Ref="C9"  Part="1"
+F 0 "C9" V 5480 6238 60  0000 L CNN
 F 1 "Конденсатор_керамический" H 5600 6050 60  0001 C CNN
-F 2 "N_RLC:Конденсатор_SMD_0603" H 5500 6150 60  0001 C CNN
+F 2 "N_RLC:Конденсатор_SMD_0603_pnp" H 5500 6150 60  0001 C CNN
 F 3 "" H 5500 6150 60  0001 C CNN
 F 4 "10мкФ/10В" V 5578 6238 50  0000 L CNN "INFO"
@@
 5V_NOISE
 $Comp
-L UAK_3-rescue:AC-DC-преобразователь_IRM-15-5-elements_2020-UAK_1-rescue-UAK_2-rescue G1
+L UAK_3-rescue:AC-DC-преобразователь_IRM-15-5-elements_2020-UAK_1-rescue-UAK_2-rescue G?
 U 1 1 5F6F4DEB
 P 4300 1500
-AR Path="/5F6F4DEB" Ref="G1"  Part="1"
+AR Path="/5F6F4DEB" Ref="G?"  Part="1"
 AR Path="/5F540B17/5F6F4DEB" Ref="G1"  Part="1"
 F 0 "G1" H 4850 1600 50  0000 C CNN
