File: UAK_3/UAK_3.sch (KiCad schematic (older format))
At the start: 57 parts, among them K1 Кнопка_FSMSM, K2 Кнопка_FSMSM, X1 Крепежное_отверстие_М3, X2 Крепежное_отверстие_М3, X3 Крепежное_отверстие_М3, X4 Крепежное_отверстие_М3, X5 Клеммник_х4, X6 Клеммник_х10

Commit message: заменен потенциометр, начал формировать BOM
Parts:
- R15: INFO (none) -> 130 Ом
- RP1: footprint MOTOR_IMPORT_OTK:резистор_подстроечный_PVZ3A334 -> N_RLC:резистор_подстроечный_3314J-1; LCSC (none) -> C36376; LINK https://www.chipdip.ru/product/3303x-3-503 -> https://lcsc.com/product-detail/Variable-Resistors_BOURNS-3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; Для заказа Резистор подстроечный 50 кОм -> Резистор подстроечный 10 кОм
- VD1: LCSC (none) -> C35501; LINK https://www.terraelectronica.ru/product/129173 -> https://lcsc.com/product-detail/Schottky-Barrier-Diodes-SBD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
- VD3: LCSC (none) -> C14308; LINK https://www.terraelectronica.ru/product/296487 -> https://lcsc.com/product-detail/Schottky-Barrier-Diodes-SBD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
- VT1, VT2, VT3, VT4: LCSC (none) -> C693370; LINK https://www.chipdip.ru/product/irlml6344trpbf -> https://lcsc.com/product-detail/MOSFET_VBsemi-Elec-IRLML634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
- X1, X2, X3, X4: LCSC (none) -> -
Other:
- note removed: "4) заменить потенциометр"
- note removed: "ПОДСВЕТКА ЛАМПЫ \n(ОТКРЫТЫЙ СТОК)"
Changed lines of the file:
@@
 EESchema Schematic File Version 4
 LIBS:UAK_3-cache
-EELAYER 29 0
+EELAYER 30 0
 EELAYER END
 $Descr A3 16535 11693
@@
 F 3 "${MOTOR_2020_LIB}\\documentation\\КрипТехно.pdf" H 13400 5800 50  0001 C CNN
 F 4 "аА0.339.471ТУ" H 13700 5450 50  0001 C CNN "TY"
-F 5 "https://www.terraelectronica.ru/product/296487" H 13500 5800 50  0001 C CNN "LINK"
+F 5 "https://lcsc.com/product-detail/Schottky-Barrier-Diodes-SBD_ON-Semiconductor-BAT54CLT1G_C14308.html/?href=jlc-SMT" H 13500 5800 50  0001 C CNN "LINK"
 F 6 "Набор диодов BAR43CFILM" H 13500 5800 50  0001 C CNN "Для заказа"
+F 7 "C14308" H 13500 5800 50  0001 C CNN "LCSC"
 	1    13500 5800
 	-1   0    0    -1
@@
 F 2 "MOTOR_VD_VT_HL:Корпус_КТ-46" H 9075 2675 60  0001 C CNN
 F 3 "" H 9000 2000 60  0001 C CNN
-F 4 "https://www.chipdip.ru/product/irlml6344trpbf" H 9025 2850 50  0001 C CNN "LINK"
+F 4 "https://lcsc.com/product-detail/MOSFET_VBsemi-Elec-IRLML6344TR_C693370.html/?href=jlc-SMT" H 9025 2850 50  0001 C CNN "LINK"
 F 5 "IRLML6344TR" H 9150 1800 50  0000 C CNN "INFO"
 F 6 "Транзистор N-канал IRLML6344TRPBF" H 9000 2000 50  0001 C CNN "Для заказа"
+F 7 "C693370" H 9000 2000 50  0001 C CNN "LCSC"
 	1    9000 2000
 	1    0    0    -1
@@
 F 3 "https://static.chipdip.ru/lib/046/DOC003046730.pdf" H 9650 1500 50  0001 C CNN
 F 4 "1А, 60В" H 9925 1050 50  0001 C CNN "INFO"
-F 5 "https://www.terraelectronica.ru/product/129173" H 9925 1175 50  0001 C CNN "LINK"
+F 5 "https://lcsc.com/product-detail/Schottky-Barrier-Diodes-SBD_MDD-Microdiode-Electronics-SS24B_C35501.html/?href=jlc-SMT" H 9925 1175 50  0001 C CNN "LINK"
 F 6 "Диод шоттки SK16 (1А 60В)" H 9750 1500 50  0001 C CNN "Для заказа"
+F 7 "C35501" H 9750 1500 50  0001 C CNN "LCSC"
 	1    9750 1500
 	0    -1   -1   0
@@
 F 5 "-" H 11000 11000 50  0001 C CNN "Для заказа"
 F 6 "-" H 11000 11000 50  0001 C CNN "LINK"
+F 7 "-" H 11000 11000 50  0001 C CNN "LCSC"
 	1    11000 11000
 	1    0    0    -1
@@
 F 5 "-" H 10500 11000 50  0001 C CNN "Для заказа"
 F 6 "-" H 10500 11000 50  0001 C CNN "LINK"
+F 7 "-" H 10500 11000 50  0001 C CNN "LCSC"
 	1    10500 11000
 	1    0    0    -1
@@
 F 5 "-" H 10000 11000 50  0001 C CNN "Для заказа"
 F 6 "-" H 10000 11000 50  0001 C CNN "LINK"
+F 7 "-" H 10000 11000 50  0001 C CNN "LCSC"
 	1    10000 11000
 	1    0    0    -1
@@
 F 5 "-" H 9500 11000 50  0001 C CNN "Для заказа"
 F 6 "-" H 9500 11000 50  0001 C CNN "LINK"
+F 7 "-" H 9500 11000 50  0001 C CNN "LCSC"
 	1    9500 11000
 	1    0    0    -1
@@
 F 0 "RP1" H 9500 4650 39  0000 C CNN
 F 1 "Резистор_подстроечный_PVA3A103" H 9900 4200 39  0001 C CNN
-F 2 "MOTOR_IMPORT_OTK:резистор_подстроечный_PVZ3A334" H 9850 4100 39  0001 C CNN
+F 2 "N_RLC:резистор_подстроечный_3314J-1" H 9850 4100 39  0001 C CNN
 F 3 "${MOTOR_2020_LIB}\\documentation\\IMPORT\\potentiometrs_PVZ.pdf" H 9300 5100 39  0001 C CNN
-F 4 "https://www.chipdip.ru/product/3303x-3-503" H 9300 5100 50  0001 C CNN "LINK"
+F 4 "https://lcsc.com/product-detail/Variable-Resistors_BOURNS-3314J-1-103E_C36376.html/?href=jlc-SMT" H 9300 5100 50  0001 C CNN "LINK"
 F 5 "10 кОм" H 9300 5100 50  0001 C CNN "INFO"
-F 6 "Резистор подстроечный 50 кОм" H 9300 5100 50  0001 C CNN "Для заказа"
+F 6 "Резистор подстроечный 10 кОм" H 9300 5100 50  0001 C CNN "Для заказа"
+F 7 "C36376" H 9300 5100 50  0001 C CNN "LCSC"
 	1    9300 5100
 	-1   0    0    -1
@@
 F 2 "MOTOR_VD_VT_HL:Корпус_КТ-46" H 9025 8725 60  0001 C CNN
 F 3 "" H 8950 8050 60  0001 C CNN
-F 4 "https://www.chipdip.ru/product/irlml6344trpbf" H 8975 8900 50  0001 C CNN "LINK"
+F 4 "https://lcsc.com/product-detail/MOSFET_VBsemi-Elec-IRLML6344TR_C693370.html/?href=jlc-SMT" H 8975 8900 50  0001 C CNN "LINK"
 F 5 "IRLML6344TR" H 9100 7850 50  0000 C CNN "INFO"
 F 6 "Транзистор N-канал IRLML6344TRPBF" H 8950 8050 50  0001 C CNN "Для заказа"
+F 7 "C693370" H 8950 8050 50  0001 C CNN "LCSC"
 	1    8950 8050
 	1    0    0    -1
@@
 F 2 "MOTOR_VD_VT_HL:Корпус_КТ-46" H 9075 4925 60  0001 C CNN
 F 3 "" H 9000 4250 60  0001 C CNN
-F 4 "https://www.chipdip.ru/product/irlml6344trpbf" H 9025 5100 50  0001 C CNN "LINK"
+F 4 "https://lcsc.com/product-detail/MOSFET_VBsemi-Elec-IRLML6344TR_C693370.html/?href=jlc-SMT" H 9025 5100 50  0001 C CNN "LINK"
 F 5 "IRLML6344TR" H 9150 4050 50  0000 C CNN "INFO"
 F 6 "Транзистор N-канал IRLML6344TRPBF" H 9000 4250 50  0001 C CNN "Для заказа"
+F 7 "C693370" H 9000 4250 50  0001 C CNN "LCSC"
 	1    9000 4250
 	1    0    0    -1
@@
 F 2 "MOTOR_VD_VT_HL:Корпус_КТ-46" H 3075 7325 60  0001 C CNN
 F 3 "" H 3000 6650 60  0001 C CNN
-F 4 "https://www.chipdip.ru/product/irlml6344trpbf" H 3025 7500 50  0001 C CNN "LINK"
+F 4 "https://lcsc.com/product-detail/MOSFET_VBsemi-Elec-IRLML6344TR_C693370.html/?href=jlc-SMT" H 3025 7500 50  0001 C CNN "LINK"
 F 5 "IRLML6344TR" H 3150 6450 50  0000 C CNN "INFO"
 F 6 "Транзистор N-канал IRLML6344TRPBF" H 3000 6650 50  0001 C CNN "Для заказа"
+F 7 "C693370" H 3000 6650 50  0001 C CNN "LCSC"
 	1    3000 6650
 	1    0    0    -1
@@
 5V
 NoConn ~ 1750 2950
-Text Notes 1750 4500 0    50   ~ 0
-4) заменить потенциометр
 $Comp
 L elements:Резистор_0,5Вт R15
@@
 F 4 "130 Ом" H 5200 7025 50  0000 C CNN "Номинал"
 F 5 "R101" H 5200 7150 50  0001 C CNN "УГО"
+F 6 "130 Ом" H 5200 7150 50  0001 C CNN "INFO"
 	1    5200 7150
 	1    0    0    -1
@@
 Text Label 6000 10050 2    50   ~ 0
 5V
-Text Notes 6200 10550 1    50   ~ 0
-ПОДСВЕТКА ЛАМПЫ \n(ОТКРЫТЫЙ СТОК)
 Text Label 6000 10200 2    50   ~ 0
 5V

Commit message: BOM переопределен по всему, кроме резисторов
Parts:
- A1: LCSC (none) -> C701341; LINK https://www.terraelectronica.ru/product/2292549 -> https://lcsc.com/product-detail/WIFI-Modules_Espressif-Syst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
- C1, C3, C4, C5, C6: LCSC (none) -> C14663; LINK https://www.terraelectronica.ru/product/1044009 -> https://lcsc.com/product-detail/Multilayer-Ceramic-Capacito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
- C2: LCSC (none) -> C313070; LINK https://www.terraelectronica.ru/product/363479 -> https://lcsc.com/product-detail/Tantalum-Capacitors_AVX-TPS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
- D1, D2, DA1, HA1, HL1, HL2, K1, K2, X5, X6, XFU1, XFU2, XP1: LCSC (none) -> -
- DD1: LCSC (none) -> C457671; LINK https://www.terraelectronica.ru/product/287011 -> https://lcsc.com/product-detail/Logic-Buffers-Drivers-Recei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
Changed lines of the file:
@@
 EESchema Schematic File Version 4
 LIBS:UAK_3-cache
-EELAYER 30 0
+EELAYER 29 0
 EELAYER END
 $Descr A3 16535 11693
@@
 F 2 "N_A:ESP32_WROVER_or_WROOM32" H 1950 1000 50  0001 C CNN
 F 3 "" H 1950 1000 50  0001 C CNN
-F 4 "https://www.terraelectronica.ru/product/2292549" H 1950 1000 50  0001 C CNN "LINK"
+F 4 "https://lcsc.com/product-detail/WIFI-Modules_Espressif-Systems-ESP32-WROOM-32E-4MB_C701341.html/?href=jlc-SMT" H 1950 1000 50  0001 C CNN "LINK"
 F 5 "ESP32-WROOM-32 [4MB]" H 1950 1000 50  0001 C CNN "Для заказа"
+F 6 "C701341" H 1950 1000 50  0001 C CNN "LCSC"
 	1    1950 1000
 	1    0    0    -1
@@
 F 4 "https://www.terraelectronica.ru/product/1087727" H 14850 4250 50  0001 C CNN "LINK"
 F 5 "Кнопка FSMSM" H 14850 4250 50  0001 C CNN "Для заказа"
+F 6 "-" H 14850 4250 50  0001 C CNN "LCSC"
 	1    14850 4250
 	1    0    0    -1
@@
 F 4 "https://www.terraelectronica.ru/product/1087727" H 14850 4750 50  0001 C CNN "LINK"
 F 5 "Кнопка FSMSM" H 14850 4750 50  0001 C CNN "Для заказа"
+F 6 "-" H 14850 4750 50  0001 C CNN "LCSC"
 	1    14850 4750
 	1    0    0    -1
@@
 F 5 "https://www.chipdip.ru/product/wf-4r" H 15000 5900 50  0001 C CNN "LINK"
 F 6 "Вилка угловая WF-4R" H 15000 5900 50  0001 C CNN "Для заказа"
+F 7 "-" H 15000 5900 50  0001 C CNN "LCSC"
 	1    15000 5900
 	-1   0    0    -1
@@
 F 3 "" H 13000 5050 60  0001 C CNN
 F 4 "0,1мкФ/50В" V 13078 5138 50  0000 L CNN "INFO"
-F 5 "https://www.terraelectronica.ru/product/1044009" H 13000 5050 50  0001 C CNN "LINK"
+F 5 "https://lcsc.com/product-detail/Multilayer-Ceramic-Capacitors-MLCC-SMD-SMT_YAGEO-CC0603KRX7R9BB104_C14663.html/?href=jlc-SMT" H 13000 5050 50  0001 C CNN "LINK"
 F 6 "Конденсатор 0603 100 нФ 50В 5%" H 13000 5050 50  0001 C CNN "Для заказа"
+F 7 "C14663" H 13000 5050 50  0001 C CNN "LCSC"
 	1    13000 5050
 	0    1    1    0
@@
 F 3 "" H 12500 5050 60  0001 C CNN
 F 4 "0,1мкФ/50В" V 12600 4500 50  0000 L CNN "INFO"
-F 5 "https://www.terraelectronica.ru/product/1044009" H 12500 5050 50  0001 C CNN "LINK"
+F 5 "https://lcsc.com/product-detail/Multilayer-Ceramic-Capacitors-MLCC-SMD-SMT_YAGEO-CC0603KRX7R9BB104_C14663.html/?href=jlc-SMT" H 12500 5050 50  0001 C CNN "LINK"
 F 6 "Конденсатор 0603 100 нФ 50В 5%" H 12500 5050 50  0001 C CNN "Для заказа"
+F 7 "C14663" H 12500 5050 50  0001 C CNN "LCSC"
 	1    12500 5050
 	0    1    1    0
@@
 F 3 "" H 13600 8000 60  0001 C CNN
 F 4 "0,1мкФ/50В" H 13400 8100 50  0000 L CNN "INFO"
-F 5 "https://www.terraelectronica.ru/product/1044009" H 13600 8000 50  0001 C CNN "LINK"
+F 5 "https://lcsc.com/product-detail/Multilayer-Ceramic-Capacitors-MLCC-SMD-SMT_YAGEO-CC0603KRX7R9BB104_C14663.html/?href=jlc-SMT" H 13600 8000 50  0001 C CNN "LINK"
 F 6 "Конденсатор 0603 100 нФ 50В 5%" H 13600 8000 50  0001 C CNN "Для заказа"
+F 7 "C14663" H 13600 8000 50  0001 C CNN "LCSC"
 	1    13600 8000
 	-1   0    0    1
@@
 F 4 "https://www.chipdip.ru/product/hpa17f" H 11025 3525 50  0001 C CNN "LINK"
 F 5 "Зуммер HPA17F" H 11100 3850 50  0001 C CNN "Для заказа"
+F 6 "-" H 11100 3850 50  0001 C CNN "LCSC"
 	1    11100 3850
 	1    0    0    -1
@@
 F 4 "-" H 10000 5500 50  0001 C CNN "Для заказа"
 F 5 "-" H 10000 5500 50  0001 C CNN "LINK"
+F 6 "-" H 10000 5500 50  0001 C CNN "LCSC"
 	1    10000 5500
 	1    0    0    -1
@@
 F 3 "" H 13600 9500 60  0001 C CNN
 F 4 "0,1мкФ/50В" H 13400 9600 50  0000 L CNN "INFO"
-F 5 "https://www.terraelectronica.ru/product/1044009" H 13600 9500 50  0001 C CNN "LINK"
+F 5 "https://lcsc.com/product-detail/Multilayer-Ceramic-Capacitors-MLCC-SMD-SMT_YAGEO-CC0603KRX7R9BB104_C14663.html/?href=jlc-SMT" H 13600 9500 50  0001 C CNN "LINK"
 F 6 "Конденсатор 0603 100 нФ 50В 5%" H 13600 9500 50  0001 C CNN "Для заказа"
+F 7 "C14663" H 13600 9500 50  0001 C CNN "LCSC"
 	1    13600 9500
 	-1   0    0    1
@@
 F 2 "N_G:Преобразователь_LM2703_SOT-23-5" H 9125 9700 50  0001 C CNN
 F 3 "https://static.chipdip.ru/lib/225/DOC000225700.pdf" H 9100 10250 50  0001 C CNN
-F 4 "https://www.terraelectronica.ru/product/287011" H 9125 9800 50  0001 C CNN "LINK"
+F 4 "https://lcsc.com/product-detail/Logic-Buffers-Drivers-Receivers-Transceivers_ON-Semiconductor-M74VHC1GT125DT1G_C457671.html/?href=jlc-SMT" H 9125 9800 50  0001 C CNN "LINK"
 F 5 "Повторитель M74VHC1GT125DT1G" H 9100 10250 50  0001 C CNN "Для заказа"
+F 6 "C457671 " H 9100 10250 50  0001 C CNN "LCSC"
 	1    9100 10250
 	1    0    0    -1
@@
 F 3 "" H 9500 9400 60  0001 C CNN
 F 4 "0,1мкФ/50В" V 9578 9488 50  0000 L CNN "INFO"
-F 5 "https://www.terraelectronica.ru/product/1044009" H 9500 9400 50  0001 C CNN "LINK"
+F 5 "https://lcsc.com/product-detail/Multilayer-Ceramic-Capacitors-MLCC-SMD-SMT_YAGEO-CC0603KRX7R9BB104_C14663.html/?href=jlc-SMT" H 9500 9400 50  0001 C CNN "LINK"
 F 6 "Конденсатор 0603 100 нФ 50В 5%" H 9500 9400 50  0001 C CNN "Для заказа"
+F 7 "C14663" H 9500 9400 50  0001 C CNN "LCSC"
 	1    9500 9400
 	0    -1   1    0
@@
 F 3 "" H 10000 9400 60  0001 C CNN
 F 4 "100мкФ/10В" V 10100 9500 50  0000 L CNN "INFO"
-F 5 "https://www.terraelectronica.ru/product/363479" V 10061 9528 50  0001 L CNN "LINK"
+F 5 "https://lcsc.com/product-detail/Tantalum-Capacitors_AVX-TPSD107K010R0050_C313070.html/?href=jlc-SMT" V 10061 9528 50  0001 L CNN "LINK"
 F 6 "Конденсатор D 100 мкФ 10В 20%" H 10000 9400 50  0001 C CNN "Для заказа"
+F 7 "C313070 " H 10000 9400 50  0001 C CNN "LCSC"
 	1    10000 9400
 	0    1    1    0
@@
 F 5 "https://www.chipdip.ru/product/kr293kp1b" H 4350 6100 50  0001 C CNN "LINK"
 F 6 "МОП-реле КР293КП1Б" H 4100 5900 50  0001 C CNN "Для заказа"
+F 7 "-" H 4100 5900 50  0001 C CNN "LCSC"
 	1    4100 5900
 	1    0    0    1
@@
 F 5 "-" H 9000 11000 50  0001 C CNN "Для заказа"
 F 6 "-" H 9000 11000 50  0001 C CNN "LINK"
+F 7 "-" H 9000 11000 50  0001 C CNN "LCSC"
 	1    9000 11000
 	1    0    0    -1
@@
 F 4 "https://www.chipdip.ru/product/kls5-266-fh-100" H 13900 1175 50  0001 C CNN "LINK"
 F 5 "Держатель KLS5-266" H 13750 1500 50  0001 C CNN "Для заказа"
+F 6 "-" H 13750 1500 50  0001 C CNN "LCSC"
 	1    13750 1500
 	1    0    0    -1
@@
 F 4 "https://www.chipdip.ru/product/kls5-266-fh-100" H 14650 1175 50  0001 C CNN "LINK"
 F 5 "Держатель KLS5-266" H 14500 1500 50  0001 C CNN "Для заказа"
+F 6 "-" H 14500 1500 50  0001 C CNN "LCSC"
 	1    14500 1500
 	-1   0    0    -1
@@
 F 5 "-" H 8500 11000 50  0001 C CNN "Для заказа"
 F 6 "-" H 8500 11000 50  0001 C CNN "LINK"
+F 7 "-" H 8500 11000 50  0001 C CNN "LCSC"
 	1    8500 11000
 	1    0    0    -1
@@
 F 2 "N_VD_HL:TFT_2.8_INCH" H 2500 8500 50  0001 C CNN
 F 3 "" H 2500 8500 50  0001 C CNN
+F 4 "-" H 2500 8500 50  0001 C CNN "LCSC"
 	1    2500 8500
 	1    0    0    -1
@@
 F 2 "N_X:Клеммник_х10_шаг3,81_15EDGRC" H 5425 9275 60  0001 C CNN
 F 3 "" H 5425 9275 60  0001 C CNN
+F 4 "-" H 6000 9000 50  0001 C CNN "LCSC"
 	1    6000 9000
 	1    0    0    -1
@@
 F 2 "N_X:Клеммник_х4_шаг3,81_15EDGRC" H 4425 9275 60  0001 C CNN
 F 3 "" H 4425 9275 60  0001 C CNN
+F 4 "-" H 5000 9000 50  0001 C CNN "LCSC"
 	1    5000 9000
 	1    0    0    -1

Commit message: подготовлены файлы для заказа в JLCPCB
Parts:
- A1: footprint N_A:ESP32_WROVER_or_WROOM32 -> N_A:ESP32_WROVER_or_WROOM32_pnp
- C1, C3, C4, C5, C6: footprint N_RLC:Конденсатор_SMD_0603 -> N_RLC:Конденсатор_SMD_0603_pnp
- C2: footprint MOTOR_RLC:Конденсатор_тантал_SMD_m7343 -> N_RLC:Конденсатор_тантал_SMD_m7343_pnp
- DD1: footprint N_G:Преобразователь_LM2703_SOT-23-5 -> N_G:SOT-23-5_pnp
- R1: renamed from R19; footprint N_RLC:Резистор_SMD_0603_0,065_Вт -> N_RLC:Резистор_SMD_0603_0,065_Вт_pnp; LCSC (none) -> C101310; LINK https://www.terraelectronica.ru/product/559067 -> https://lcsc.com/product-detail/Chip-Resistor-Surface-Mount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
- R10: renamed from R25; footprint N_RLC:Резистор_SMD_0603_0,065_Вт -> N_RLC:Резистор_SMD_0603_0,065_Вт_pnp; LCSC (none) -> C101310; LINK https://www.terraelectronica.ru/product/559067 -> https://lcsc.com/product-detail/Chip-Resistor-Surface-Mount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
- R11: renamed from R1; footprint N_RLC:Резистор_SMD_0603_0,065_Вт -> N_RLC:Резистор_SMD_0603_0,065_Вт_pnp; LCSC (none) -> C101310; LINK https://www.terraelectronica.ru/product/559067 -> https://lcsc.com/product-detail/Chip-Resistor-Surface-Mount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
- R12: renamed from R2; footprint N_RLC:Резистор_SMD_0603_0,065_Вт -> N_RLC:Резистор_SMD_0603_0,065_Вт_pnp; LCSC (none) -> C101310; LINK https://www.terraelectronica.ru/product/559067 -> https://lcsc.com/product-detail/Chip-Resistor-Surface-Mount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
- R13: renamed from R3; footprint N_RLC:Резистор_SMD_0603_0,065_Вт -> N_RLC:Резистор_SMD_0603_0,065_Вт_pnp; LCSC (none) -> C101310; LINK https://www.terraelectronica.ru/product/559067 -> https://lcsc.com/product-detail/Chip-Resistor-Surface-Mount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
- R14: renamed from R4; footprint N_RLC:Резистор_SMD_0603_0,065_Вт -> N_RLC:Резистор_SMD_0603_0,065_Вт_pnp; LCSC (none) -> C510290; LINK https://www.terraelectronica.ru/product/562124 -> https://lcsc.com/product-detail/Chip-Resistor-Surface-Mount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
- R15: renamed from R5; footprint N_RLC:Резистор_SMD_0603_0,065_Вт -> N_RLC:Резистор_SMD_0603_0,065_Вт_pnp; LCSC (none) -> C510290; LINK https://www.terraelectronica.ru/product/562124 -> https://lcsc.com/product-detail/Chip-Resistor-Surface-Mount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
- R16: renamed from R6; footprint N_RLC:Резистор_SMD_0603_0,065_Вт -> N_RLC:Резистор_SMD_0603_0,065_Вт_pnp; LCSC (none) -> C510290; LINK https://www.terraelectronica.ru/product/562124 -> https://lcsc.com/product-detail/Chip-Resistor-Surface-Mount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
- R17: renamed from R23; footprint N_RLC:Резистор_SMD_1206-0,25_Вт -> N_RLC:Резистор_SMD_1206-0,25_Вт_pnp; INFO 4,7 кОм -> 1 кОм; LCSC (none) -> C830401; LINK https://www.terraelectronica.ru/product/2782734 -> https://lcsc.com/product-detail/Chip-Resistor-Surface-Mount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
- R18: renamed from R7; footprint N_RLC:Резистор_SMD_0603_0,065_Вт -> N_RLC:Резистор_SMD_0603_0,065_Вт_pnp; LCSC (none) -> C510290; LINK https://www.terraelectronica.ru/product/562124 -> https://lcsc.com/product-detail/Chip-Resistor-Surface-Mount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
- R19: renamed from R8; footprint N_RLC:Резистор_SMD_0603_0,065_Вт -> N_RLC:Резистор_SMD_0603_0,065_Вт_pnp; LCSC (none) -> C510290; LINK https://www.terraelectronica.ru/product/562124 -> https://lcsc.com/product-detail/Chip-Resistor-Surface-Mount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
- R2: renamed from R20; footprint N_RLC:Резистор_SMD_0603_0,065_Вт -> N_RLC:Резистор_SMD_0603_0,065_Вт_pnp; LCSC (none) -> C510290; LINK https://www.terraelectronica.ru/product/562124 -> https://lcsc.com/product-detail/Chip-Resistor-Surface-Mount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
- R20: renamed from R9; footprint N_RLC:Резистор_SMD_0603_0,065_Вт -> N_RLC:Резистор_SMD_0603_0,065_Вт_pnp; LCSC (none) -> C510290; LINK https://www.terraelectronica.ru/product/562124 -> https://lcsc.com/product-detail/Chip-Resistor-Surface-Mount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
- R21: renamed from R10; footprint N_RLC:Резистор_SMD_0603_0,065_Вт -> N_RLC:Резистор_SMD_0603_0,065_Вт_pnp; LCSC (none) -> C510290; LINK https://www.terraelectronica.ru/product/562124 -> https://lcsc.com/product-detail/Chip-Resistor-Surface-Mount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
- R22: renamed from R11; footprint N_RLC:Резистор_SMD_0603_0,065_Вт -> N_RLC:Резистор_SMD_0603_0,065_Вт_pnp; LCSC (none) -> C101310; LINK https://www.terraelectronica.ru/product/559067 -> https://lcsc.com/product-detail/Chip-Resistor-Surface-Mount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
- R23: renamed from R12; footprint N_RLC:Резистор_SMD_0603_0,065_Вт -> N_RLC:Резистор_SMD_0603_0,065_Вт_pnp; LCSC (none) -> C101310; LINK https://www.terraelectronica.ru/product/559067 -> https://lcsc.com/product-detail/Chip-Resistor-Surface-Mount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
- R24: renamed from R13; footprint N_RLC:Резистор_SMD_0603_0,065_Вт -> N_RLC:Резистор_SMD_0603_0,065_Вт_pnp; LCSC (none) -> C101310; LINK https://www.terraelectronica.ru/product/559067 -> https://lcsc.com/product-detail/Chip-Resistor-Surface-Mount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
- R25: renamed from R14; footprint N_RLC:Резистор_SMD_0603_0,065_Вт -> N_RLC:Резистор_SMD_0603_0,065_Вт_pnp; LCSC (none) -> C101310; LINK https://www.terraelectronica.ru/product/559067 -> https://lcsc.com/product-detail/Chip-Resistor-Surface-Mount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
- R3: renamed from R21; footprint N_RLC:Резистор_SMD_0603_0,065_Вт -> N_RLC:Резистор_SMD_0603_0,065_Вт_pnp; LCSC (none) -> C336847; LINK https://www.terraelectronica.ru/product/569439 -> https://lcsc.com/product-detail/Others_PANASONIC-ERJ3RBD150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
- R4: renamed from R15; footprint N_RLC:Резистор_SMD_2010-0,5_Вт -> N_RLC:Резистор_SMD_2010-0,5_Вт_pnp; LCSC (none) -> C406994; LINK (none) -> https://lcsc.com/product-detail/Chip-Resistor-Surface-Mount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
- R5: renamed from R16; footprint N_RLC:Резистор_SMD_0603_0,065_Вт -> N_RLC:Резистор_SMD_0603_0,065_Вт_pnp; LCSC (none) -> C101310; LINK https://www.terraelectronica.ru/product/559067 -> https://lcsc.com/product-detail/Chip-Resistor-Surface-Mount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
- R6: renamed from R17; footprint N_RLC:Резистор_SMD_0603_0,065_Вт -> N_RLC:Резистор_SMD_0603_0,065_Вт_pnp; LCSC (none) -> C101310; LINK https://www.terraelectronica.ru/product/559067 -> https://lcsc.com/product-detail/Chip-Resistor-Surface-Mount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
- R7: renamed from R18; footprint N_RLC:Резистор_SMD_0603_0,065_Вт -> N_RLC:Резистор_SMD_0603_0,065_Вт_pnp; LCSC (none) -> C101310; LINK https://www.terraelectronica.ru/product/559067 -> https://lcsc.com/product-detail/Chip-Resistor-Surface-Mount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
- R8: renamed from R22; footprint N_RLC:Резистор_SMD_0603_0,065_Вт -> N_RLC:Резистор_SMD_0603_0,065_Вт_pnp; LCSC (none) -> C101310; LINK https://www.terraelectronica.ru/product/559067 -> https://lcsc.com/product-detail/Chip-Resistor-Surface-Mount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
- R9: renamed from R24; footprint N_RLC:Резистор_SMD_0603_0,065_Вт -> N_RLC:Резистор_SMD_0603_0,065_Вт_pnp; LCSC (none) -> C101310; LINK https://www.terraelectronica.ru/product/559067 -> https://lcsc.com/product-detail/Chip-Resistor-Surface-Mount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
- RP1: footprint N_RLC:резистор_подстроечный_3314J-1 -> N_RLC:резистор_подстроечный_3314J-1_pnp
- VD1: footprint N_VD_HL:Диод_SMB -> N_VD_HL:Диод_SMB_pnp; symbol UAK_3-rescue:Диод_шоттки_SK16-elements_2020-UAK_0-rescue-UAK_1-rescue-UAK_2-rescue -> elements_2020:Диод_шоттки_SK16
- VD2: renamed from VD3; footprint MOTOR_VD_VT_HL:Корпус_КТ-46 -> N_DD:Корпус_КТ-46_pnp
- VT1: renamed from VT4; footprint MOTOR_VD_VT_HL:Корпус_КТ-46 -> N_DD:Корпус_КТ-46_pnp
- VT2: renamed from VT1; footprint MOTOR_VD_VT_HL:Корпус_КТ-46 -> N_DD:Корпус_КТ-46_pnp
- VT3: renamed from VT2; footprint MOTOR_VD_VT_HL:Корпус_КТ-46 -> N_DD:Корпус_КТ-46_pnp
- VT4: renamed from VT3; footprint MOTOR_VD_VT_HL:Корпус_КТ-46 -> N_DD:Корпус_КТ-46_pnp
- renumbered D2 to D1, D1 to D2, HL2 to HL1, HL1 to HL2, X5 to X1, X6 to X2, X1 to X3, X2 to X4, X3 to X5, X4 to X6
Connections:
- net 5V: now also VD1.1; no longer VD1.2
- net D_OUT_1: now also VD1.2; no longer VD1.1
